File: kicad/greenhouse.kicad_sch (KiCad schematic)
At the start: 21 parts, among them J1 LED 16x2, J2 moisture sensor, J3 fan, J4 dht11, J5 Conn_01x04, Q1 IRLZ44N, U1 ESP-12F, U3 AMS1117-3.3

Commit message: ыыыыыыыыыыыыыыы
Parts:
- removed J1: LED 16x2, symbol Connector_Generic:Conn_01x04
- removed U3: AMS1117-3.3, Package_TO_SOT_SMD:SOT-223-3_TabPin2, symbol Regulator_Linear:AMS1117-3.3
- added D1: SS34, Diode_SMD:D_SMA, symbol Device:D_Schottky
- added J6: Barrel_Jack_Switch, Connector_BarrelJack:BarrelJack_Horizontal, symbol Connector:Barrel_Jack_Switch
- added L1: 33uH, Inductor_SMD:L_12x12mm_H8mm, symbol Device:L
- added U2: LM2596S-3.3, Package_TO_SOT_SMD:TO-263-5_TabPin3, symbol Regulator_Switching:LM2596S-3.3
- C1: footprint Capacitor_SMD:C_0603_1608Metric_Pad1.08x0.95mm_HandSolder -> Capacitor_THT:CP_Radial_D5.0mm_P2.00mm
- C2: footprint Capacitor_SMD:C_0603_1608Metric_Pad1.08x0.95mm_HandSolder -> Capacitor_THT:C_Disc_D5.0mm_W2.5mm_P2.50mm
- C3: value 100nF -> 220uF; footprint Capacitor_SMD:C_0603_1608Metric_Pad1.08x0.95mm_HandSolder -> Capacitor_THT:CP_Radial_D5.0mm_P2.00mm
- C4: value 100uF -> 220uF; footprint (none) -> Capacitor_THT:CP_Radial_D5.0mm_P2.00mm
- C5: footprint (none) -> Capacitor_THT:C_Disc_D5.0mm_W2.5mm_P2.50mm
- J1: renamed from pump1; footprint TerminalBlock_Phoenix:TerminalBlock_Phoenix_MKDS-1-2-3.81_1x02_P3.81mm_Horizontal -> TerminalBlock_Phoenix:TerminalBlock_Phoenix_MKDS-3-2-5.08_1x02_P5.08mm_Horizontal
- J2: footprint Connector_PinHeader_1.00mm:PinHeader_1x03_P1.00mm_Horizontal -> Connector_PinHeader_2.54mm:PinHeader_1x03_P2.54mm_Vertical
- J3: footprint (none) -> Connector_PinHeader_2.54mm:PinHeader_1x03_P2.54mm_Vertical
- J4: value dht11 -> DHT11; footprint (none) -> Connector_PinHeader_2.54mm:PinHeader_1x03_P2.54mm_Vertical
- J5: footprint (none) -> Connector_PinHeader_2.54mm:PinHeader_1x04_P2.54mm_Vertical
- R1, R2, R3, R4: footprint Resistor_SMD:R_0603_1608Metric_Pad0.98x0.95mm_HandSolder -> Resistor_SMD:R_0805_2012Metric_Pad1.20x1.40mm_HandSolder
- R5, R6, R7: footprint (none) -> Resistor_SMD:R_0805_2012Metric_Pad1.20x1.40mm_HandSolder
Connections:
- net +3.3V: now also C1.1, C2.1, C4.1, C5.2, J2.2 (Pin_2), L1.2, U2.4 (FB); no longer C1.2, C2.2, C5.1, J2.1 (Pin_1), J3.2 (Pin_2)
- net GND: now also C1.2, C2.2, C5.1, J2.1 (Pin_1), J3.2 (Pin_2), D1.2 (A), J6.2, U2.3 (GND), U2.5 (~{ON}/OFF); no longer C1.1, C2.1, C5.2, J2.2 (Pin_2), J3.3 (Pin_3)
- net +5V renamed +12V
- net +12V: now also J3.3 (Pin_3), J6.1, U2.1 (VIN); no longer C4.1
- new net: D1.1 (K), L1.1, U2.2 (OUT)
- no-connect marks 6 -> 10
Other:
- moved on the sheet: C1, C2

Commit message: 123
Parts:
- removed C5: 100nF, Capacitor_THT:C_Disc_D5.0mm_W2.5mm_P2.50mm, symbol Device:C
- added H1, H2, H3, H4: MountingHole, MountingHole:MountingHole_2.2mm_M2_Pad, symbol Mechanical:MountingHole
Connections:
- net +3.3V: now also J1.1 (Pin_1); no longer J1.2 (Pin_2)
- net GND: now also J5.3 (Pin_3); no longer J5.1 (Pin_1)
- net at U1.21 (GPIO3/RXD): now also J5.2 (Pin_2); no longer J5.3 (Pin_3)
- net at U1.22 (GPIO1/TXD): now also J5.1 (Pin_1); no longer J5.2 (Pin_2)
- net at Q1.2 (D): now also J1.2 (Pin_2); no longer J1.1 (Pin_1)
Other:
- moved on the sheet: J1, R2

Commit message: 123
Parts:
- added J7: relay, Connector_PinHeader_2.54mm:PinHeader_1x02_P2.54mm_Vertical, symbol Connector_Generic:Conn_01x02
Connections:
- net GND: now also J7.1 (Pin_1)
- net at U1.6 (GPIO12): now also J7.2 (Pin_2)
- no-connect marks 10 -> 9
Changed lines of the file:
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@@
 	)
 	(no_connect
-		(at 114.3 74.93)
-	)
-	(no_connect
 		(at 83.82 80.01)
 	)
@@
 	(wire
 		(pts
+			(xy 114.3 74.93) (xy 132.08 74.93)
+		)
+		(stroke
+			(width 0)
+			(type default)
+		)
+	)
+	(wire
+		(pts
 			(xy 119.38 95.25) (xy 118.11 95.25)
 		)
@@
 	(wire
 		(pts
+			(xy 129.54 72.39) (xy 132.08 72.39)
+		)
+		(stroke
+			(width 0)
+			(type default)
+		)
+	)
+	(wire
+		(pts
 			(xy 130.81 104.14) (xy 132.08 104.14)
 		)
@@
 	)
 	(symbol
+		(lib_id "Connector_Generic:Conn_01x02")
+		(at 137.16 72.39 0)
+		(unit 1)
+		(exclude_from_sim no)
+		(in_bom yes)
+		(on_board yes)
+		(dnp no)
+		(fields_autoplaced yes)
+		(property "Reference" "J7"
+			(at 139.7 72.3899 0)
+			(effects
+				(font
+					(size 1.27 1.27)
+				)
+				(justify left)
+			)
+		)
+		(property "Value" "relay"
+			(at 139.7 74.9299 0)
+			(effects
+				(font
+					(size 1.27 1.27)
+				)
+				(justify left)
+			)
+		)
+		(property "Footprint" "Connector_PinHeader_2.54mm:PinHeader_1x02_P2.54mm_Vertical"
+			(at 137.16 72.39 0)
+			(effects
+				(font
+					(size 1.27 1.27)
+				)
+				(hide yes)
+			)
+		)
+		(property "Datasheet" "~"
+			(at 137.16 72.39 0)
+			(effects
+				(font
+					(size 1.27 1.27)
+				)
+				(hide yes)
+			)
+		)
+		(property "Description" "Generic connector, single row, 01x02, script generated (kicad-library-utils/schlib/autogen/connector/)"
+			(at 137.16 72.39 0)
+			(effects
+				(font
+					(size 1.27 1.27)
+				)
+				(hide yes)
+			)
+		)
+		(pin "2"
+		)
+		(pin "1"
+		)
+		(instances
+			(project ""
+				(path "/a3c52171-5c7d-4cff-ba66-31b186ab2256"
+					(reference "J7")
+					(unit 1)
+				)
+			)
+		)
+	)
+	(symbol
 		(lib_id "Device:R")
 		(at 114.3 40.64 90)
@@
 					(unit 1)
 				)
+			)
+		)
+	)
+	(symbol
+		(lib_id "power:GND")
+		(at 129.54 72.39 270)
+		(unit 1)
+		(exclude_from_sim no)
+		(in_bom yes)
+		(on_board yes)
+		(dnp no)
+		(fields_autoplaced yes)
+		(property "Reference" "#PWR07"
+			(at 123.19 72.39 0)
+			(effects
+				(font
+					(size 1.27 1.27)
+				)
+				(hide yes)
+			)
+		)
+		(property "Value" "GND"
+			(at 125.73 72.3899 90)
+			(effects
+				(font
+					(size 1.27 1.27)
+				)
+				(justify right)
+			)
+		)
+		(property "Footprint" ""
+			(at 129.54 72.39 0)
+			(effects
+				(font
+					(size 1.27 1.27)
+				)
+				(hide yes)
+			)
+		)
+		(property "Datasheet" ""
+			(at 129.54 72.39 0)
+			(effects
+				(font
+					(size 1.27 1.27)
+				)
+				(hide yes)
+			)
+		)
+		(property "Description" "Power symbol creates a global label with name \"GND\" , ground"
+			(at 129.54 72.39 0)
+			(effects
+				(font
+					(size 1.27 1.27)
+				)
+				(hide yes)
+			)
+		)
+		(pin "1"
+		)
+		(instances
+			(project ""
+				(path "/a3c52171-5c7d-4cff-ba66-31b186ab2256"
+					(reference "#PWR07")
+					(unit 1)
+				)
